File: Hardware/Binary_Blaster.brd (EAGLE design)
At the start: 86.4 x 69.8 mm, 26 parts

Commit message: cleaned up part values on buttons
Parts:
- S3, S4, S5, S6: value SWITCH-MOMENTARY-LEDEZ -> (none)
Changed lines of the file:
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@@
 <element name="U$3" library="SparkFun" package="OSHW-LOGO-S" value="OSHW-LOGOS" x="41.275" y="64.135" rot="MR0"/>
 <element name="U$7" library="Testing" package="DIL28-3_KEYED-14" value="AVR-MEGA8-P-KEYED-14" x="43.18" y="53.34"/>
-<element name="S3" library="SparkFun-Electromechanical" package="TACTILE-PTH-LED-12MM-EZ" value="SWITCH-MOMENTARY-LEDEZ" x="20.32" y="8.89"/>
-<element name="S4" library="SparkFun-Electromechanical" package="TACTILE-PTH-LED-12MM-EZ" value="SWITCH-MOMENTARY-LEDEZ" x="35.56" y="8.89"/>
-<element name="S5" library="SparkFun-Electromechanical" package="TACTILE-PTH-LED-12MM-EZ" value="SWITCH-MOMENTARY-LEDEZ" x="50.8" y="8.89"/>
-<element name="S6" library="SparkFun-Electromechanical" package="TACTILE-PTH-LED-12MM-EZ" value="SWITCH-MOMENTARY-LEDEZ" x="66.04" y="8.89"/>
+<element name="S3" library="SparkFun-Electromechanical" package="TACTILE-PTH-LED-12MM-EZ" value="" x="20.32" y="8.89"/>
+<element name="S4" library="SparkFun-Electromechanical" package="TACTILE-PTH-LED-12MM-EZ" value="" x="35.56" y="8.89"/>
+<element name="S5" library="SparkFun-Electromechanical" package="TACTILE-PTH-LED-12MM-EZ" value="" x="50.8" y="8.89"/>
+<element name="S6" library="SparkFun-Electromechanical" package="TACTILE-PTH-LED-12MM-EZ" value="" x="66.04" y="8.89"/>
 <element name="FRAME1" library="SparkFun-Aesthetics" package="CREATIVE_COMMONS" value="FRAME-LETTER" x="-135.362121875" y="0"/>
 <element name="LOGO1" library="SparkFun-Aesthetics" package="SFE-NEW-WEBLOGO" value="LOGO-SFENEW" x="33.782" y="63.373"/>

Commit message: Added LED polarity swap trick
Still V03
Parts:
- added JP10, JP11, JP12, JP13, JP14, JP4, JP8, JP9: (no value), SparkFun-Passives:SJ_3
Connections:
- net GND: now also JP10.1, JP11.2, JP11.3, JP12.1, JP13.2, JP13.3, JP14.1, JP4.2, JP4.3, JP8.1, JP9.2, JP9.3
- net LED0: now also JP4.1, JP8.2, JP8.3
- net LED1: now also JP10.2, JP10.3, JP9.1
- net LED2: now also JP11.1, JP12.2, JP12.3
- net LED3: now also JP13.1, JP14.2, JP14.3
Routing:
- net LED0: track 43.7 -> 70.5 mm, vias 0 -> 1
- net LED3: track 41.7 -> 65.5 mm, vias 0 -> 1
- net LED1: track 51.4 -> 72.6 mm, vias 0 -> 1
- net LED2: track 65.4 -> 86.0 mm, vias 0 -> 1
- net GND: track 217.4 -> 235.6 mm, vias 0 -> 4
- net BUTTON3: track 108.1 -> 114.6 mm
- net D: track 102.9 -> 98.9 mm
- net BUTTON2: track 99.0 -> 102.4 mm
- net BUTTON1: track 96.6 -> 94.0 mm
- net BUTTON0: track 88.2 -> 86.0 mm
- net N$4: vias 0 -> 2
- net N$2: vias 0 -> 1

Commit message: V10
-changed bottom copper version to "v10"
-added "pete lewis" to designed by on board tname layer
-changed version to "10" on schematic
Parts:
- moved FRAME1 148.9 mm to (13.2, -8.89)
Other:
- board text added: "Pete Lewis"
- board text added: "V10"
- board text removed: "V03"
